Commit message: as1 updates

File: minimal_robot_description/minimal_robot_description.urdf (robot description, URDF)
Before this commit: robot one_DOF_robot, 3 links, 2 joints
Links:
- added link link3, mass 1; collision cylinder length=0.5 radius=0.05; visual cylinder length=0.5 radius=0.05
Joints:
- added joint joint2: type continuous, parent link2, child link3, origin xyz=0 0 0.7 rpy=0 0 0, axis 0 1 0
